File: examples/eagle6/TSOC-ESP8266-EM/TSOC-ESP8266-EM/revisions/TSOC-ESP8266-EM.sch (EAGLE design)
At the start: 21 parts, among them Q1 MMBT2222A, U1 ESP8266-12-12W

Commit message: update modules
Parts:
- removed U$16: TSOC-32-BB, thingSoC:TSOC-32-BB
- added C3, C4: 0.1uF, PatternAgents-ProtoPads:CAP0402-CAP
- added JP1: (no value), PatternAgents-ProtoPads:JMP-2-NO-0402
- added LED1: LED-TRICOLOR, SparkFun-LED:LED-TRICOLOR
- added R15: 0.01, PatternAgents-ProtoPads:RESISTOR0402
- added R16, R17, R18: 560, PatternAgents-ProtoPads:RESISTOR0402
- added TSOC: TSOC-24-BB, thingSoC:TSOC-24-BB
- added U$11: PA_LOGO_SYMMED, PatternAgents-Logos:PA_LOGO_SYMMED
- added U2: EEPROM-I2CSMD, SparkFun-DigitalIC:EEPROM-I2CSMD
- added U3: TMP102, SparkFun-Sensors:TMP102
- added U4: ATECC108, SparkFun-DigitalIC:ATECC108
- U$19, U$20: value TSOC-LOGO-SMALL -> TSOC-LOGO-MED; device thingSoC:TSOC-LOGO-SMALL -> thingSoC:TSOC-LOGO-MED
Connections:
- net RESET renamed !RST
- removed net !DBG: U$16.!JDBG
- removed net A0: R8.2, U$16.!RI
- new net !DCD: TSOC.!DCD
- new net !RI: TSOC.!RI
- new net 3V3I: C1.1, C2.1, R15.2, TSOC.3V3
- new net ADC_RAW: JP1.2, R8.2
- new net BLU: LED1.BLU, R16.2
- new net GRN: LED1.GRN, R17.2
- new net RED: LED1.RED, R18.2
- net !CTS: now also TSOC.!CTS; no longer U$16.!CTS, U$16.JTDI
- net !DSR: now also TSOC.!DSR; no longer U$16.!DSR
- net !DTR: now also TSOC.!DTR; no longer U$16.!DTR, U$16.!JRST
- net !RTS: now also TSOC.!RTS; no longer U$16.!RTS, U$16.JTDO
- net 3V3: now also C3.2, C4.2, JP1.1, LED1.A, R15.1, U2.A0, U2.A1, U2.A2, U2.VCC, U3.VCC, U4.VCC; no longer C1.1, C2.1, U$16.3V3, U$16.VTARG
- net GND: now also C3.1, C4.1, TSOC.AGND, TSOC.GND, U2.VSS, U2.WP, U3.ADD0, U3.GND; no longer U$16.AGND, U$16.GND, U$16.GNDJ
- net GPIO0: now also R18.1, TSOC.SS2
- net GPIO1: now also TSOC.RXD; no longer U$16.JTCK, U$16.RXD
- net GPIO12: now also TSOC.MISO; no longer U$16.MISO
- net GPIO13: now also TSOC.MOSI; no longer U$16.MOSI
- net GPIO14: now also TSOC.SCK; no longer U$16.SCK
- net GPIO15: now also TSOC.!CS; no longer U$16.!CS
- net GPIO16: now also TSOC.IO1; no longer U$16.!DCD
- net GPIO2: now also TSOC.SS1; no longer U$16.IO2
- net GPIO3: now also TSOC.TXD; no longer U$16.JTMS, U$16.TXD
- net GPIO4: now also R16.1, TSOC.SDA, U2.SDA, U3.SDA, U4.SDA; no longer U$16.SDA
- net GPIO5: now also R17.1, TSOC.SCL, U2.SCL, U3.SCL, U4.SCL; no longer U$16.SCL
Other:
- note added: "I2C Temp Sensor"
- note added: "NOTE: 1) Connect JP1 for Volts or Temp. Measurement 2) R8 is 10K resistor for Volt Measurement 3) R8 is 10K Thermistor for Temp, Measurement 4) Connect External Sensor to JP1-Pin2"
- note added: "NVSRAM FM24V10 (128K x 8 bits SRAM)"
- note added: "Normal Booting -------------- CH_PD (High) GPIO0 (High) GPIO2 (High) GPIO15 (Low)"
- note removed: "1) Add Power LED 2) Add GPIO5/LED 3) Add Sensors (Temp/Light/etc)"
- note removed: "@PatternAgents"
- note removed: "Normal Booting --------------------- CH_PD (High) GPIO0 (High) GPIO2 (High) GPIO15 (Low)"
- moved on the sheet: C1, C2, Q1G$1, Q1G$2, R1, R10, R11, R12, R13, R14, R2, R3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
