File: examples/eagle6/TSOC-ESP8266-EM/TSOC-ESP8266-EM/TSOC-ESP8266-EM.brd (EAGLE design)
At the start: 38.4 x 26.4 mm, 33 parts, among them Q1 MMBT2222A, U1 ESP8266-12-12W, U2 EEPROM-I2CSMD, U3 TMP102, U4 ATECC108

Commit message: update modules
Parts:
- moved C3 24.9 mm to (2.29, 5.08)
- moved C4 24.9 mm to (29.2, 16.5)
- moved R12 24.9 mm to (8.89, 19.6)
- moved U1 24.9 mm to (27.2, 13.5)
- moved C1 24.9 mm to (3.30, 23.4)
- moved C2 24.9 mm to (3.30, 21.8)
- moved JP1 24.9 mm to (4.83, 17.8)
- moved LED1 24.9 mm to (4.57, 8.89)
- moved Q1 24.9 mm to (9.14, 13.5)
- moved R1 24.9 mm to (5.08, 15.7)
- moved R10 24.9 mm to (14.0, 14.2)
- moved R11 24.9 mm to (12.2, 18.3)
- moved R13 24.9 mm to (8.64, 17.0)
- moved R14 24.9 mm to (12.2, 15.7)
- moved R15 24.9 mm to (3.30, 20.3)
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Routing:
- net GND: track 131.7 -> 132.4 mm

Commit message: embedded module updates
Parts:
- moved C3 0.76 mm to (3.05, 5.08)
Routing:
- net 3V3: track 108.5 -> 109.3 mm
- net GND: track 132.4 -> 133.2 mm
Changed lines of the file:
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@@
 <setting verticaltext="up"/>
 </settings>
-<grid distance="10" unitdist="mil" unit="mm" style="lines" multiple="1" display="yes" altdistance="0.025" altunitdist="inch" altunit="inch"/>
+<grid distance="10" unitdist="mil" unit="mil" style="lines" multiple="1" display="yes" altdistance="0.025" altunitdist="inch" altunit="inch"/>
 <layers>
 <layer number="1" name="Top" color="4" fill="1" visible="yes" active="yes"/>
@@
 <attribute name="VALUE" x="2.794" y="12.319" size="0.4064" layer="28" rot="MR180"/>
 </element>
-<element name="C3" library="PatternAgents-ProtoPads" package="0402-CAP" value="0.1uF" x="2.286" y="5.08" rot="MR90"/>
+<element name="C3" library="PatternAgents-ProtoPads" package="0402-CAP" value="0.1uF" x="3.048" y="5.08" rot="MR90"/>
 <element name="U3" library="SparkFun-Sensors" package="SOT563" value="TMP102" x="8.128" y="11.938" smashed="yes" rot="MR90">
 <attribute name="PROD_ID" value="IC-09303" x="8.128" y="11.938" size="1.778" layer="28" rot="MR90" display="off"/>
@@
 <wire x1="3.429" y1="14.3002" x2="2.159" y2="14.3002" width="0.254" layer="16"/>
 <wire x1="4.699" y1="14.3002" x2="3.429" y2="14.3002" width="0.254" layer="16"/>
-<wire x1="2.286" y1="5.66" x2="2.286" y2="7.112" width="0.254" layer="16"/>
 <wire x1="2.286" y1="7.112" x2="2.286" y2="8.9408" width="0.254" layer="16"/>
 <wire x1="2.286" y1="8.9408" x2="2.159" y2="9.0678" width="0.254" layer="16"/>
@@
 <wire x1="28.448" y1="18.542" x2="28.448" y2="16.692" width="0.254" layer="16"/>
 <wire x1="28.448" y1="16.692" x2="28.63" y2="16.51" width="0.254" layer="16"/>
+<wire x1="3.048" y1="5.66" x2="3.048" y2="6.858" width="0.254" layer="16"/>
+<wire x1="3.048" y1="6.858" x2="2.794" y2="7.112" width="0.254" layer="16"/>
+<wire x1="2.794" y1="7.112" x2="2.032" y2="7.112" width="0.254" layer="16"/>
 </signal>
 <signal name="GND">
@@
 <wire x1="5.969" y1="16.129" x2="5.842" y2="16.256" width="0.254" layer="16"/>
 <wire x1="5.842" y1="16.256" x2="1.016" y2="16.256" width="0.254" layer="16"/>
-<wire x1="2.286" y1="4.5" x2="2.286" y2="2.794" width="0.254" layer="16"/>
-<wire x1="2.286" y1="2.794" x2="1.778" y2="2.286" width="0.254" layer="16"/>
 <polygon width="0.254" layer="16" spacing="0.254" pour="hatch" isolate="0.254" orphans="yes">
 <vertex x="0" y="0.254"/>
@@
 <wire x1="12.192" y1="8.89" x2="12.374" y2="8.636" width="0.1778" layer="1"/>
 <wire x1="12.192" y1="8.89" x2="12.28849375" y2="8.89" width="0.1778" layer="1"/>
-<wire x1="12.446" y1="8.89" x2="12.374" y2="8.636" width="0.1778" layer="1"/>
 <wire x1="12.446" y1="9.906" x2="12.374" y2="9.906" width="0.1778" layer="1"/>
 <wire x1="12.446" y1="9.906" x2="12.446" y2="9.820478125" width="0.1778" layer="1"/>
 <wire x1="12.446" y1="8.636" x2="12.374" y2="8.636" width="0.1778" layer="1"/>
 <wire x1="12.446" y1="8.636" x2="12.4595" y2="8.72151875" width="0.1778" layer="1"/>
+<wire x1="1.778" y1="2.286" x2="2.54" y2="2.286" width="0.254" layer="16"/>
+<wire x1="2.54" y1="2.286" x2="3.048" y2="2.794" width="0.254" layer="16"/>
+<wire x1="3.048" y1="2.794" x2="3.048" y2="4.5" width="0.254" layer="16"/>
+<wire x1="12.446" y1="8.89" x2="12.374" y2="8.636" width="0.1778" layer="1"/>
 </signal>
 <signal name="GPIO1">
